Commit message: refactor: rename robot model files and replace iron-x naming with robot

File: models/model robot/urdf/robot.urdf (robot description, URDF)
Before this commit: robot IRON-X PRO TESR THESIS v.1, 8 links, 7 joints
Links:
- link base_link: geometry collision mesh filename=package://robot_model/meshes/base_link.STL; visual mesh filename=package://robot_model/meshes/base_link.STL
- link camera_link: geometry collision mesh filename=package://robot_model/meshes/camera_link.STL; visual mesh filename=package://robot_model/meshes/camera_link.STL
- link imu_link: geometry collision mesh filename=package://robot_model/meshes/imu_link.STL; visual mesh filename=package://robot_model/meshes/imu_link.STL
- link left_back_link: geometry collision mesh filename=package://robot_model/meshes/left_back_link.STL; visual mesh filename=package://robot_model/meshes/left_back_link.STL
- link left_front_link: geometry collision mesh filename=package://robot_model/meshes/left_front_link.STL; visual mesh filename=package://robot_model/meshes/left_front_link.STL
- link lidar_link: geometry collision mesh filename=package://robot_model/meshes/lidar_link.STL; visual mesh filename=package://robot_model/meshes/lidar_link.STL
- link right_back_link: geometry collision mesh filename=package://robot_model/meshes/right_back_link.STL; visual mesh filename=package://robot_model/meshes/right_back_link.STL
- link right_front_link: geometry collision mesh filename=package://robot_model/meshes/right_front_link.STL; visual mesh filename=package://robot_model/meshes/right_front_link.STL

Commit message: Fix lidar_joint to fixed type and add Gazebo Harmonic plugins and sensors

File: models/model robot/urdf/robot.urdf (robot description, URDF)
Before this commit: robot robot_model, 9 links, 8 joints
Joints:
- joint lidar_joint: axis 0 0 -1 -> (none); type continuous -> fixed
