Commit message: refactor: rename simulation package iron_x to robot and clean up paths

File: simulation/robot/urdf/robot.urdf (robot description, URDF)
Before this commit: robot pro, 10 links, 9 joints
Links:
- link base_link: geometry collision mesh filename=package://robot/meshes/base_link.STL; visual mesh filename=package://robot/meshes/base_link.STL
- link camera_link: geometry collision mesh filename=package://robot/meshes/camera_link.STL; visual mesh filename=package://robot/meshes/camera_link.STL
- link imu_link: geometry collision mesh filename=package://robot/meshes/imu_link.STL; visual mesh filename=package://robot/meshes/imu_link.STL
- link left_back_link: geometry collision mesh filename=package://robot/meshes/left_back_link.STL; visual mesh filename=package://robot/meshes/left_back_link.STL
- link left_front_link: geometry collision mesh filename=package://robot/meshes/left_front_link.STL; visual mesh filename=package://robot/meshes/left_front_link.STL
- link lidar_link: geometry collision mesh filename=package://robot/meshes/lidar_link.STL; visual mesh filename=package://robot/meshes/lidar_link.STL
- link right_back_link: geometry collision mesh filename=package://robot/meshes/right_back_link.STL; visual mesh filename=package://robot/meshes/right_back_link.STL
- link right_front_link: geometry collision mesh filename=package://robot/meshes/right_front_link.STL; visual mesh filename=package://robot/meshes/right_front_link.STL

Commit message: Update simulation packages for ROS 2 Jazzy and Gazebo Harmonic

File: simulation/robot/urdf/robot.urdf (robot description, URDF)
Before this commit: robot pro, 10 links, 9 joints
Joints:
- joint lidar_joint: axis 0 0 -1 -> (none)
